File: uaefi.kicad_pcb (KiCad board)
At the start: 4 copper layers, 133.2 x 100 mm, 142 parts, among them J23 2-6447232-3, J25 2-6447232-3, J6 Conn_01x06, J7 Conn_01x05_Male, J8 USB_B_Mini, J9 USB_C, M1 Module-power_12and5V-0.3, M2 Module-knock-0.2, M3 Module-vr-discrete-0.5, M4 Module-vr-max9924-0.1, M5 Module-wbo-0.5, M6 Module:mega-mcu100/0.3, M7 Module-can-0.1, P1 Pad, P15 Pad, P16 Pad, P17 Pad, P18 Pad, P2 Pad, P3 Pad, P4 Pad, P5 Pad, P6 Pad, P7 Pad, P8 Pad, Q10 ISL9V3040D3ST, Q11 ISL9V3040D3ST, Q12 ISL9V3040D3ST, Q7 ISL9V3040D3ST, Q8 ISL9V3040D3ST, Q9 ISL9V3040D3ST, U1 TLE9201SG, U10 VNLD5160TR-E, U11 VNLD5160TR-E, U2 TLE9201SG, U3 MPX4/MPXH6400_MAP, U4 MAX31855KASA, U5 JDY-33, U6 VNLD5160TR-E, U7 VNLD5160TR-E, U8 VNLD5160TR-E, U9 VNLD5160TR-E

Commit message: mkn
mnj
Parts:
- moved BT1 33.2 mm to (175.2, 134.5)
- moved C13 33.2 mm to (99.9, 145.0)
- moved C16 33.2 mm to (97.8, 150.5)
- moved C17 33.2 mm to (99.8, 150.5)
- moved C18 33.2 mm to (101.8, 150.5)
- moved C21 33.2 mm to (97.8, 154.5)
- moved C22 33.2 mm to (99.8, 154.5)
- moved C23 33.2 mm to (101.8, 154.5)
- moved C26 33.2 mm to (106.8, 154.5)
- moved C29 33.2 mm to (138.7, 82.9)
- moved C30 33.2 mm to (140.4, 77.4)
- moved C31 33.2 mm to (142.8, 86.5)
- moved C33 33.2 mm to (180.2, 126.0)
- moved D1 33.2 mm to (171.2, 144.0)
- moved D8 33.2 mm to (138.7, 80.4)
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
Commit message: a
Parts:
- removed G1: RUSEFI_LOGO, kicad6-libraries:rusefi_logo
- removed G2: LOGO, hellen-one-common:LOGO
- removed G3, G4: PROTO_AREA, hellen-one-common:PROTO_AREA
- removed P1, P2: Pad, hellen-one-common:PAD-TH
- removed Q10, Q11, Q12, Q7, Q8, Q9: ISL9V3040D3ST, Package_TO_SOT_SMD:TO-252-2
- removed R17, R18, R19, R23, R24, R25: 22, hellen-one-common:R0603
- removed R20, R21, R22, R26, R27, R28: 0, Resistor_SMD:R_2512_6332Metric
- D3, D5, R1, R10, R11, U7: moved to B.Cu
- F10, F5, F6, F7, F8, F9: moved to F.Cu
- moved R1 78.4 mm to (57.8, 130.1), turned to 90 degrees
- moved R40 67.8 mm to (113.6, 75.3), turned to 90 degrees
- moved R37 62.3 mm to (115.7, 75.3), turned to -90 degrees
- moved F10 55.7 mm to (110.6, 125.7), turned to 0 degrees
- moved D4 48.6 mm to (87.7, 128.4), turned to 0 degrees
- moved R13 47.9 mm to (99.5, 132.5)
- moved R12 47.8 mm to (99.5, 129.0)
- moved U8 47.6 mm to (95.0, 130.0)
- moved D5 42.5 mm to (87.7, 130.9), turned to 0 degrees
- moved R33 37.0 mm to (93.2, 102.2), turned to 180 degrees
- moved R38 36.2 mm to (145.4, 72.7)
- moved R32 33.3 mm to (87.7, 115.8), turned to 0 degrees
- moved H1 33.2 mm to (53.5, 63.5)
- moved H2 33.2 mm to (53.5, 156.5)
- moved R35 33.0 mm to (145.4, 74.6), turned to 180 degrees
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Connections:
- F1 pad 1: /12V_KEY -> 12V_KEY
- F10 pad 1: Net-(F10-Pad1) -> /OUT_IGN6
- F5 pad 1: Net-(F5-Pad1) -> /OUT_IGN2
- F6 pad 1: Net-(F6-Pad1) -> /OUT_IGN1
- F7 pad 1: Net-(F7-Pad1) -> /OUT_IGN3
- F8 pad 1: Net-(F8-Pad1) -> /OUT_IGN4
- F9 pad 1: Net-(F9-Pad1) -> /OUT_IGN5
- J23 pad 1: unconnected-(J23-Pad1) -> /OUT_LS2
- J23 pad 10: unconnected-(J23-Pad10) -> /OUT_LS1
- J23 pad 11: unconnected-(J23-Pad11) -> /OUT_IGN2
- J23 pad 12: unconnected-(J23-Pad12) -> /OUT_IGN4
- J23 pad 13: unconnected-(J23-Pad13) -> /OUT_IGN6
- J23 pad 14: unconnected-(J23-Pad14) -> /OUT_INJ6
- J23 pad 15: unconnected-(J23-Pad15) -> /OUT_INJ4
- J23 pad 16: unconnected-(J23-Pad16) -> /OUT_INJ2
- J23 pad 17: unconnected-(J23-Pad17) -> 12V_KEY
- J23 pad 18: unconnected-(J23-Pad18) -> /VR_MAX9924+
- J23 pad 19: unconnected-(J23-Pad19) -> CAN2L
- J23 pad 2: unconnected-(J23-Pad2) -> /OUT_IGN1
- J23 pad 20: unconnected-(J23-Pad20) -> CAN2H
- J23 pad 21: unconnected-(J23-Pad21) -> +5VP
- J23 pad 22: unconnected-(J23-Pad22) -> +5VP
- J23 pad 23: unconnected-(J23-Pad23) -> +5VP
- J23 pad 24: unconnected-(J23-Pad24) -> +5VP
- J23 pad 25: unconnected-(J23-Pad25) -> +12V
- J23 pad 26: unconnected-(J23-Pad26) -> /VR_DISCRETE+
- J23 pad 27: unconnected-(J23-Pad27) -> /VR_DISCRETE-
- J23 pad 28: unconnected-(J23-Pad28) -> /VR_MAX9924-
- J23 pad 29: unconnected-(J23-Pad29) -> GND
- J23 pad 3: unconnected-(J23-Pad3) -> /OUT_IGN3
- J23 pad 30: unconnected-(J23-Pad30) -> GND
- J23 pad 31: unconnected-(J23-Pad31) -> /OUT_DC2-
- J23 pad 32: unconnected-(J23-Pad32) -> /OUT_DC2+
- J23 pad 33: unconnected-(J23-Pad33) -> /OUT_DC1-
- J23 pad 34: /OUT_DC1- -> /OUT_DC1+
- J23 pad 4: unconnected-(J23-Pad4) -> /OUT_IGN5
- J23 pad 5: unconnected-(J23-Pad5) -> /OUT_INJ5
- J23 pad 6: unconnected-(J23-Pad6) -> /OUT_INJ3
- J23 pad 7: unconnected-(J23-Pad7) -> /OUT_INJ1
- J23 pad 8: unconnected-(J23-Pad8) -> /OUT_LS3
- J23 pad 9: unconnected-(J23-Pad9) -> /OUT_LS4
- J25 pad 1: unconnected-(J25-Pad1) -> /IN_BUTTON1
- J25 pad 10: unconnected-(J25-Pad10) -> /IN_BUTTON2
- J25 pad 11: unconnected-(J25-Pad11) -> +5VA
- J25 pad 12: unconnected-(J25-Pad12) -> +5VA
- J25 pad 13: unconnected-(J25-Pad13) -> +5VA
- J25 pad 14: unconnected-(J25-Pad14) -> /IN_TPS2
- J25 pad 15: unconnected-(J25-Pad15) -> /IN_PPS2
- J25 pad 16: unconnected-(J25-Pad16) -> /IN_HALL1
- J25 pad 17: unconnected-(J25-Pad17) -> /IN_HALL3
- J25 pad 18: unconnected-(J25-Pad18) -> /IN_TPS1
- J25 pad 19: unconnected-(J25-Pad19) -> /IN_FLEX
- J25 pad 2: unconnected-(J25-Pad2) -> +5VA
- J25 pad 20: unconnected-(J25-Pad20) -> /IN_MAP
- J25 pad 21: unconnected-(J25-Pad21) -> /IN_AUX1
- J25 pad 22: unconnected-(J25-Pad22) -> /IN_AUX2
- J25 pad 23: unconnected-(J25-Pad23) -> /IN_BUTTON3
- J25 pad 25: unconnected-(J25-Pad25) -> /OUT_LS_HOT2
- J25 pad 26: unconnected-(J25-Pad26) -> /IN_PPS1
- J25 pad 27: unconnected-(J25-Pad27) -> /IN_KNOCK_RAW
- J25 pad 28: unconnected-(J25-Pad28) -> /IN_IAT
- J25 pad 29: unconnected-(J25-Pad29) -> /IN_CLT
- J25 pad 3: unconnected-(J25-Pad3) -> GNDA
- J25 pad 30: unconnected-(J25-Pad30) -> /CAN+
- J25 pad 31: unconnected-(J25-Pad31) -> /CAN-
- J25 pad 34: unconnected-(J25-Pad34) -> /OUT_LS_HOT1
- J25 pad 4: unconnected-(J25-Pad4) -> GNDA
- J25 pad 5: unconnected-(J25-Pad5) -> GNDA
- J25 pad 6: unconnected-(J25-Pad6) -> GNDA
- J25 pad 7: unconnected-(J25-Pad7) -> GNDA
- J25 pad 8: unconnected-(J25-Pad8) -> /IN_AUX3
- J25 pad 9: unconnected-(J25-Pad9) -> /IN_HALL2
- M7 pad S1: Net-(M7-CANL) -> CAN2L
- M7 pad S2: Net-(M7-CANH) -> CAN2H
Routing:
- net +12V_RAW: track 250.7 -> 88.9 mm
- net /CAN-: track 100.8 -> 237.1 mm, vias 0 -> 1
- net /CAN+: track 102.6 -> 228.6 mm, vias 0 -> 1
- net /IN_CLT: track 46.2 -> 165.3 mm, vias 0 -> 1
- net /IN_KNOCK_RAW: track 4.49 -> 121.8 mm
- net /IN_IAT: track 42.6 -> 158.9 mm, vias 0 -> 1
- net +5VP: track 199.7 -> 91.8 mm, vias 3 -> 0
- net +5VA: track 171.8 -> 277.5 mm, vias 6 -> 9
- net /IN_TPS1: track 39.1 -> 144.7 mm
- net /IN_FLEX: track 45.1 -> 146.5 mm
- net /IN_PPS1: track 47.4 -> 148.3 mm
- net /IN_MAP: track 40.3 -> 130.1 mm
- net Net-(F10-Pad1): track 85.2 -> 0.00 mm, vias 2 -> 0
- net /VR_DISCRETE-: track 8.50 -> 90.5 mm
- net /IN_AUX1: track 49.8 -> 131.4 mm
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Other:
- board text removed: "+ EGT -"
- board text removed: "Always looking for C/C++/PHP/Java developers https://rusefi.com/s/mission"
- board text removed: "BT2"
- board text removed: "COMMUNITY SUPPORT ECU"
- board text removed: "DC1-"
- board text removed: "DC2-"
- board text removed: "Ignition logic level outputs by default to control dumb coils remove R20-R22, R26-R28 and populate Q7-Q12"

Commit message: A
AAA
Connections:
- J25 pad 1: /IN_BUTTON1 -> /IN_TPS1
- J25 pad 10: /IN_BUTTON2 -> /IN_PPS1
- J25 pad 11: +5VA -> /IN_FLEX
- J25 pad 12: +5VA -> /IN_BUTTON1
- J25 pad 13: +5VA -> /IN_AUX1
- J25 pad 18: /IN_TPS1 -> /EGT+
- J25 pad 19: /IN_FLEX -> /EGT-
- J25 pad 2: +5VA -> /IN_BUTTON2
- J25 pad 20: /IN_MAP -> /IN_KNOCK_RAW
- J25 pad 21: /IN_AUX1 -> IN_MAP
- J25 pad 24: unconnected-(J25-Pad24) -> /WBO_Rtrim
- J25 pad 26: /IN_PPS1 -> /WBO_Heater
- J25 pad 27: /IN_KNOCK_RAW -> /IN_IAT
- J25 pad 28: /IN_IAT -> /IN_CLT
- J25 pad 29: /IN_CLT -> /CAN+
- J25 pad 30: /CAN+ -> /CAN-
- J25 pad 31: /CAN- -> /WBO_Vm
- J25 pad 32: unconnected-(J25-Pad32) -> /WBO_Ip
- J25 pad 33: unconnected-(J25-Pad33) -> /WBO_Un
- M6 pad S13: /IN_MAP -> IN_MAP
Routing:
- net /WBO_Un: track 1.68 -> 185.0 mm, vias 0 -> 1
- net /WBO_Rtrim: track 2.19 -> 182.5 mm, vias 0 -> 1
- net /WBO_Ip: track 2.87 -> 172.8 mm, vias 0 -> 1
- net /WBO_Vm: track 2.76 -> 170.6 mm, vias 0 -> 1
- net /WBO_Heater: track 3.40 -> 149.2 mm
- net /IN_MAP: track 130.1 -> 0.00 mm
- net IN_MAP: track 0.00 -> 129.4 mm
- net /EGT-: track 6.33 -> 79.7 mm
- net /EGT+: track 10.1 -> 81.6 mm
- net +5VA: track 277.5 -> 226.1 mm
- net /IN_TPS1: track 144.7 -> 136.1 mm
- net /IN_FLEX: track 146.5 -> 140.8 mm
- net /IN_BUTTON1: track 122.0 -> 127.0 mm
- net /IN_AUX1: track 131.4 -> 126.5 mm
- net /IN_PPS1: track 148.3 -> 143.9 mm
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Other:
- board text added: "BUTTON 1"
- board text added: "BUTTON 2"
- board text removed: "1"
- board text removed: "10"
- board text removed: "11"
- board text removed: "12"
- board text removed: "12V"
- board text removed: "16"
- board text removed: "18"
- board text removed: "20"
- board text removed: "3"
- board text removed: "3.3"
- board text removed: "4"
- board text removed: "5"
- board text removed: "5V"
- board text removed: "6"
- board text removed: "8"
- board text removed: "9"
- board text removed: "9924+"
- board text removed: "9924-"
- board text removed: "A"
- board text removed: "AUX1"
- board text removed: "AUX2"
- board text removed: "AUX3"
- board text removed: "B"
- board text removed: "BT1"
- board text removed: "BT3"
- board text removed: "BTN1"
- board text removed: "BTN2"
- board text removed: "BTN3"
- board text removed: "C"
- board text removed: "CLT"
- board text removed: "D"
- board text removed: "DC1+"
- board text removed: "DC2+"
- board text removed: "DISCRETE+"
- board text removed: "DISCRETE-"
- board text removed: "E"
- board text removed: "FLEX"
- board text removed: "GND"
- board text removed: "GNDA"
- board text removed: "H"
- board text removed: "H CAN L"
- board text removed: "HALL1"
- board text removed: "HALL2"
- board text removed: "HALL3"
- board text removed: "Heater"
- board text removed: "IAT"
- board text removed: "IGN1"
- board text removed: "IGN2"
- board text removed: "IGN3"
- board text removed: "IGN4"
- board text removed: "IGN5"
- board text removed: "IGN6"
- board text removed: "INJ1"
- board text removed: "INJ2"
- board text removed: "INJ3"
- board text removed: "INJ4"
- board text removed: "INJ5"
- board text removed: "INJ6"
- board text removed: "KNOCK"
- board text removed: "L CAN H"
- board text removed: "LS1"
- board text removed: "LS2"
- board text removed: "LS3"
- board text removed: "LS4"
- board text removed: "LSH1"
- board text removed: "LSH2"
- board text removed: "MAP"
- board text removed: "PPS1"
- board text removed: "PPS2"
- board text removed: "Rtrim"
- board text removed: "TPS1"
- board text removed: "TPS2"
- board text removed: "Un"
- board text removed: "VIGN"
- board text removed: "Vm"
- board text removed: "https://rusefi.com/s/uaefi"
