File: uaefi.kicad_pcb (KiCad board)
At the start: 4 copper layers, 133.2 x 100 mm, 118 parts, among them J23 2-6447232-3, J25 2-6447232-3, J6 Conn_01x06, J7 Conn_01x05_Male, J8 USB_B_Mini, J9 USB_C, M1 Module-power_12and5V-0.3, M2 Module-knock-0.2, M3 Module-vr-discrete-0.5, M4 Module-vr-max9924-0.1, M5 Module-wbo-0.5, M6 Module:mega-mcu100/0.3, M7 Module-can-0.1, P15 Pad, P16 Pad, P17 Pad, P18 Pad, P3 Pad, P4 Pad, P5 Pad, P6 Pad, P7 Pad, P8 Pad, U1 TLE9201SG, U10 VNLD5160TR-E, U11 VNLD5160TR-E, U2 TLE9201SG, U3 MPX4/MPXH6400_MAP, U4 MAX31855KASA, U5 JDY-33, U6 VNLD5160TR-E, U7 VNLD5160TR-E, U8 VNLD5160TR-E, U9 VNLD5160TR-E

Commit message: Final?
Parts:
- moved J23 2.81 mm to (75.1, 134.3)
- moved C27 2.63 mm to (147.6, 94.9)
- moved C28 2.63 mm to (139.6, 77.4)
- moved C32 2.63 mm to (147.2, 86.5)
- moved J6 2.63 mm to (184.0, 122.1)
- moved M5 2.63 mm to (185.2, 120.4)
- moved R5 2.63 mm to (142.7, 98.2)
- moved U5 2.63 mm to (178.5, 138.9)
- moved C1 2.63 mm to (89.9, 141.0)
- moved C10 2.63 mm to (97.9, 145.0)
- moved C2 2.63 mm to (91.9, 141.0)
- moved C3 2.63 mm to (93.9, 141.0)
- moved C4 2.63 mm to (95.9, 141.0)
- moved C5 2.63 mm to (97.9, 141.0)
- moved C6 2.63 mm to (89.9, 145.0)
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Routing:
- net /WBO_Vm: track 170.6 -> 166.7 mm
- net /VR_DISCRETE-: track 90.8 -> 94.0 mm
- net 12V_KEY: track 53.7 -> 51.5 mm
- net /IN_FLEX: track 140.8 -> 138.9 mm
- net /IGN3: track 81.3 -> 79.8 mm
- net /OUT_IGN6: track 44.2 -> 45.4 mm, vias 1 -> 0
- net /OUT_IGN5: track 41.2 -> 42.4 mm
- net /IN_AUX1: track 126.5 -> 125.3 mm
- net +3.3V: track 108.0 -> 106.9 mm
- net /IN_HALL1: track 118.2 -> 119.2 mm
- net /WBO_Un: track 185.0 -> 186.1 mm
- net /WBO_Rtrim: track 182.5 -> 183.5 mm
- net /OUT_LS2: track 39.0 -> 38.0 mm, vias 1 -> 0
- net /OUT_LS1: track 47.9 -> 46.9 mm, vias 1 -> 0
- net /OUT_INJ5: track 39.2 -> 38.2 mm
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Other:
- board size 133.2 x 100 mm -> 135.7 x 100 mm
- board text removed: "G"

Commit message: Final marking
Parts:
- added G***: LOGO, LOGO 45X17:LOGO 45X17, F.Cu at (96.5, 110.7)
- added G***: LOGO, LOGO 45X17:LOGO 45X17, B.Cu at (116.2, 70.1)
Routing:
- net GND: track 1.50 -> 6.62 mm
Other:
- board text added: "4.7Kohm = VR2- AS HALL SENSOR INPUT"
- board text added: "6X6+WBO ECU V1.01 SN: FW:"
- board text added: "A"
- board text added: "B"
- board text removed: "Ip"
- board text removed: "L"
- board text removed: "UAEFI rev. E"

Commit message: Prod Candidate 1
Parts:
- added G***: LOGO, rohs:rohs, F.Cu at (177.7, 81.7)
- added G***: LOGO, CE:CE 10x7,2, F.Cu at (177.7, 73.9)
Other:
- board text added: "Disclaimer: The owner/user is solely responsible for ensuring compliance with all applicable local regulations for on-road use. The manufacturer/designer assumes no liability for improper use."

Commit message: tt
Parts:
- removed C1, C10, C14, C15, C16, C17, C18, C19, C2, C20, C21, C22, C23, C3, C4, C5, C6, C7, C8, C9: 10u, hellen-one-common:C0805
- removed C11, C24, C29, C31: 100n, hellen-one-common:C0603
- removed C12, C13, C25, C26, C28, C30: 10n, hellen-one-common:C0603
- removed C32: 1u, hellen-one-common:C0603
- removed D8: NUP2105L, Package_TO_SOT_SMD:SOT-23
- removed F3, F4: 12H1500D, hellen-one-common:PAD-1206-PAD
- removed L1, L2: 470R@100MHz, Inductor_SMD:L_0603_1608Metric
- removed M2: Module-knock-0.2, hellen-one-knock-0.2:knock
- removed M7: Module-can-0.1, hellen-one-can-0.1:can
- removed P15, P16, P17, P18: Pad, hellen-one-common:PAD-TH
- removed R14, R9: 4.7k, hellen-one-common:R0603
- removed U1, U2: TLE9201SG, Package_SO:Infineon_PG-DSO-12-11
- removed U4: MAX31855KASA, Package_SO:SOIC-8_3.9x4.9mm_P1.27mm
Connections:
- M6 pad E6: Net-(M6-SPI2_CS_/_CAN2_RX_(PB12)) -> unconnected-(M6-SPI2_CS_/_CAN2_RX_(PB12)-PadE6)
- M6 pad E7: Net-(M6-SPI2_SCK_/_CAN2_TX_(PB13)) -> unconnected-(M6-SPI2_SCK_/_CAN2_TX_(PB13)-PadE7)
- M6 pad E8: /DC1_DIS -> unconnected-(M6-SPI2_MISO_(PB14)-PadE8)
- M6 pad E9: /DC2_DIR -> unconnected-(M6-SPI2_MOSI_(PB15)-PadE9)
- M6 pad N10: /SCK3 -> unconnected-(M6-SPI3_SCK_(PC10)-PadN10)
- M6 pad N11: /MISO3 -> unconnected-(M6-SPI3_MISO_(PC11)-PadN11)
- M6 pad N12: /PG_5VP -> unconnected-(M6-SPI3_MOSI_(PC12)-PadN12)
- M6 pad N9: /EGT/SPI_CS -> unconnected-(M6-SPI3_CS_(PA15)-PadN9)
Routing:
- net /IN_KNOCK_RAW: track 120.9 -> 0.00 mm
- net +3.3VA: track 169.4 -> 51.2 mm, vias 6 -> 2
- net /EGT/SPI_CS: track 111.5 -> 0.00 mm, vias 1 -> 0
- net /SCK3: track 107.3 -> 0.00 mm, vias 1 -> 0
- net +3.3V: track 106.9 -> 0.00 mm, vias 8 -> 0
- net /MISO3: track 104.7 -> 0.00 mm, vias 1 -> 0
- net /EGT+: track 81.6 -> 0.00 mm
- net /EGT-: track 79.7 -> 0.00 mm
- net /OUT_DC2+: track 67.0 -> 0.00 mm, vias 1 -> 0
- net /DC1_DIR: track 63.7 -> 0.00 mm, vias 1 -> 0
- net /DC1_PWM: track 60.7 -> 0.00 mm, vias 2 -> 0
- net /OUT_DC2-: track 60.2 -> 0.00 mm
- net CAN2H: track 59.7 -> 0.00 mm
- net CAN2L: track 58.5 -> 0.00 mm
- net /DC2_DIR: track 58.1 -> 0.00 mm, vias 2 -> 0
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- removed copper zone on B.Cu, net /DC Driver 1/PWR
- removed copper zone on B.Cu, net /DC Driver 2/PWR
Other:
- board text added: "660 WBO ECU V1.01 SN: FW:"
- board text added: "BUTTON 3"
- board text removed: "6X6+WBO ECU V1.01 SN: FW:"
- board text removed: "CAN2"

Commit message: a
b
Parts:
- added C1: 10u, hellen-one-common:C0805, B.Cu at (89.9, 141.0)
- added C10: 10u, hellen-one-common:C0805, B.Cu at (97.9, 145.0)
- added C11: 100n, hellen-one-common:C0603, F.Cu at (87.4, 142.7)
- added C12: 10n, hellen-one-common:C0603, F.Cu at (87.4, 145.8)
- added C13: 10n, hellen-one-common:C0603, F.Cu at (102.5, 145.0)
- added C14: 10u, hellen-one-common:C0805, B.Cu at (96.4, 150.5)
- added C15: 10u, hellen-one-common:C0805, B.Cu at (98.4, 150.5)
- added C16: 10u, hellen-one-common:C0805, B.Cu at (100.4, 150.5)
- added C17: 10u, hellen-one-common:C0805, B.Cu at (102.4, 150.5)
- added C18: 10u, hellen-one-common:C0805, B.Cu at (104.4, 150.5)
- added C19: 10u, hellen-one-common:C0805, B.Cu at (96.4, 154.5)
- added C2: 10u, hellen-one-common:C0805, B.Cu at (91.9, 141.0)
- added C20: 10u, hellen-one-common:C0805, B.Cu at (98.4, 154.5)
- added C21: 10u, hellen-one-common:C0805, B.Cu at (100.4, 154.5)
- added C22: 10u, hellen-one-common:C0805, B.Cu at (102.4, 154.5)
- added C23: 10u, hellen-one-common:C0805, B.Cu at (104.4, 154.5)
- added C24: 100n, hellen-one-common:C0603, F.Cu at (93.4, 151.0)
- added C25: 10n, hellen-one-common:C0603, F.Cu at (93.4, 154.5)
- added C26: 10n, hellen-one-common:C0603, F.Cu at (109.4, 154.5)
- added C28: 10n, hellen-one-common:C0603, B.Cu at (139.6, 77.4)
- added C29: 100n, hellen-one-common:C0603, B.Cu at (141.3, 82.9)
- added C3: 10u, hellen-one-common:C0805, B.Cu at (93.9, 141.0)
- added C30: 10n, hellen-one-common:C0603, B.Cu at (143.0, 77.4)
- added C31: 100n, hellen-one-common:C0603, B.Cu at (145.4, 86.5)
- added C32: 1u, hellen-one-common:C0603, B.Cu at (147.2, 86.5)
- added C4: 10u, hellen-one-common:C0805, B.Cu at (95.9, 141.0)
- added C5: 10u, hellen-one-common:C0805, B.Cu at (97.9, 141.0)
- added C6: 10u, hellen-one-common:C0805, B.Cu at (89.9, 145.0)
- added C7: 10u, hellen-one-common:C0805, B.Cu at (91.9, 145.0)
- added C8: 10u, hellen-one-common:C0805, B.Cu at (93.9, 145.0)
- added C9: 10u, hellen-one-common:C0805, B.Cu at (95.9, 145.0)
- added D8: NUP2105L, Package_TO_SOT_SMD:SOT-23, B.Cu at (141.3, 80.4)
- added F3: 12H1500D, hellen-one-common:PAD-1206-PAD, F.Cu at (106.4, 143.0)
- added F4: 12H1500D, hellen-one-common:PAD-1206-PAD, F.Cu at (104.2, 143.0)
- added L1: 470R@100MHz, Inductor_SMD:L_0603_1608Metric, B.Cu at (142.3, 75.0)
- added L2: 470R@100MHz, Inductor_SMD:L_0603_1608Metric, B.Cu at (140.3, 75.0)
- added M2: Module-knock-0.2, hellen-one-knock-0.2:knock, F.Cu at (162.8, 77.9)
- added M7: Module-can-0.1, hellen-one-can-0.1:can, F.Cu at (116.4, 105.3)
- added P15: Pad, hellen-one-common:PAD-TH, F.Cu at (91.3, 148.5)
- added P16: Pad, hellen-one-common:PAD-TH, F.Cu at (93.9, 148.5)
- added P17: Pad, hellen-one-common:PAD-TH, F.Cu at (88.8, 148.5)
- added P18: Pad, hellen-one-common:PAD-TH, F.Cu at (108.8, 149.0)
- added R14: 4.7k, hellen-one-common:R0603, F.Cu at (109.4, 151.6)
- added R9: 4.7k, hellen-one-common:R0603, F.Cu at (102.5, 142.0)
- added U1: TLE9201SG, Package_SO:Infineon_PG-DSO-12-11, F.Cu at (94.8, 142.5)
- added U2: TLE9201SG, Package_SO:Infineon_PG-DSO-12-11, F.Cu at (101.4, 151.9)
- added U4: MAX31855KASA, Package_SO:SOIC-8_3.9x4.9mm_P1.27mm, B.Cu at (141.3, 88.2)
Connections:
- M6 pad E6: unconnected-(M6-SPI2_CS_/_CAN2_RX_(PB12)-PadE6) -> Net-(M6-SPI2_CS_/_CAN2_RX_(PB12))
- M6 pad E7: unconnected-(M6-SPI2_SCK_/_CAN2_TX_(PB13)-PadE7) -> Net-(M6-SPI2_SCK_/_CAN2_TX_(PB13))
- M6 pad E8: unconnected-(M6-SPI2_MISO_(PB14)-PadE8) -> /DC1_DIS
- M6 pad E9: unconnected-(M6-SPI2_MOSI_(PB15)-PadE9) -> /DC2_DIR
- M6 pad N10: unconnected-(M6-SPI3_SCK_(PC10)-PadN10) -> /SCK3
- M6 pad N11: unconnected-(M6-SPI3_MISO_(PC11)-PadN11) -> /MISO3
- M6 pad N12: unconnected-(M6-SPI3_MOSI_(PC12)-PadN12) -> /PG_5VP
- M6 pad N9: unconnected-(M6-SPI3_CS_(PA15)-PadN9) -> /EGT/SPI_CS
Routing:
- net /IN_KNOCK_RAW: track 0.00 -> 120.9 mm
- net +3.3VA: track 51.2 -> 169.4 mm, vias 2 -> 6
- net /EGT/SPI_CS: track 0.00 -> 111.5 mm, vias 0 -> 1
- net /SCK3: track 0.00 -> 107.3 mm, vias 0 -> 1
- net +3.3V: track 0.00 -> 106.9 mm, vias 0 -> 8
- net /MISO3: track 0.00 -> 104.7 mm, vias 0 -> 1
- net /EGT+: track 0.00 -> 81.6 mm
- net /EGT-: track 0.00 -> 79.7 mm
- net /OUT_DC2+: track 0.00 -> 67.0 mm, vias 0 -> 1
- net /DC1_DIR: track 0.00 -> 63.7 mm, vias 0 -> 1
- net /DC1_PWM: track 0.00 -> 60.7 mm, vias 0 -> 2
- net /OUT_DC2-: track 0.00 -> 60.2 mm
- net CAN2H: track 0.00 -> 59.7 mm
- net CAN2L: track 0.00 -> 58.5 mm
- net /DC2_DIR: track 0.00 -> 58.1 mm, vias 0 -> 2
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- added copper zone on B.Cu, net /DC Driver 1/PWR
- added copper zone on B.Cu, net /DC Driver 2/PWR
Other:
- board text added: "CAN2"
- board text added: "xECU 862 V1.02 SN: FW:"
- board text removed: "660 WBO ECU V1.01 SN: FW:"
- board text removed: "BUTTON 3"
