File: uaefi.kicad_sch (KiCad schematic)
At the start: 72 parts, among them J1 Conn_02x02_Odd_Even, J1 USB_B_Mini, J1 USB_C, J10 5569-16A2, J11 Conn_02x02_Odd_Even, J12 Conn_02x02_Odd_Even, J13 Conn_02x02_Odd_Even, J14 Conn_02x02_Odd_Even, J15 Conn_02x02_Odd_Even, J16 Conn_02x02_Odd_Even, J17 Conn_01x06, J17 Conn_02x02_Odd_Even, J18 Conn_02x02_Odd_Even, J19 Conn_02x02_Odd_Even, J2 5569-20A2, J20 Conn_02x02_Odd_Even, J21 Conn_02x02_Odd_Even, J22 Conn_02x02_Odd_Even, J24 Conn_02x02_Odd_Even, J3 5569-06A2, J4 5569-08A2, J5 5569-18A2, J5 Conn_01x05_Male, M1 Module-power_12and5V-0.3, M3 Module-knock-0.2, M3 Module-vr-discrete-0.5, M4 Module-vr-max9924-0.1, M5 Module-wbo-0.5, M6 Module:mega-mcu100/0.3, M7 Module-can-0.1, P1 Pad, P2 Pad, P3 Pad, P4 Pad, P5 Pad, P6 Pad, P7 Pad, P8 Pad, U4 JDY-33

Commit message: a
c
Parts:
- added J23, J25: 2-6447232-3, kicad6-libraries:TE 2-6447232-3, symbol 2-6447232-3:2-6447232-3
Connections:
- net OUT_DC1-: now also J23.34

Commit message: a
Parts:
- removed G1: RUSEFI_LOGO, kicad6-libraries:rusefi_logo, symbol rusefi_logo:RUSEFI_LOGO
- removed G2: LOGO, hellen-one-common:LOGO, symbol hellen-one-common:LOGO
- removed P1, P2: Pad, hellen-one-common:PAD-TH, symbol hellen-one-common:Pad
- added M8: Module-mega-mcu144-0.7, hellen-one-mega-mcu144-0.7:mega-mcu144, symbol Hellen 144:Module-mega-mcu144-0.7
- G3, G4: now left out of the parts list
Connections:
- net +12V: now also J23.25
- net +5VA: now also J25.11, J25.12, J25.13, J25.2
- net +5VP: now also J23.21, J23.22, J23.23, J23.24
- net 12V_KEY: now also J23.17
- net CAN+: now also J25.30
- net CAN-: now also J25.31
- net GND: now also J23.29, J23.30
- net GNDA: now also J25.3, J25.4, J25.5, J25.6, J25.7
- net IN_AUX1: now also J25.21
- net IN_AUX2: now also J25.22
- net IN_AUX3: now also J25.8
- net IN_BUTTON1: now also J25.1
- net IN_BUTTON2: now also J25.10
- net IN_BUTTON3: now also J25.23
- net IN_CLT: now also J25.29
- net IN_FLEX: now also J25.19
- net IN_HALL1: now also J25.16
- net IN_HALL2: now also J25.9
- net IN_HALL3: now also J25.17
- net IN_IAT: now also J25.28
- net IN_KNOCK_RAW: now also J25.27
- net IN_MAP: now also J25.20
- net IN_PPS1: now also J25.26
- net IN_PPS2: now also J25.15
- net IN_TPS1: now also J25.18
- net IN_TPS2: now also J25.14
- net OUT_DC1+: now also J23.34
- net OUT_DC1-: now also J23.33; no longer J23.34
- net OUT_DC2+: now also J23.32
- net OUT_DC2-: now also J23.31
- net OUT_IGN1: now also J23.2
- net OUT_IGN2: now also J23.11
- net OUT_IGN3: now also J23.3
- net OUT_IGN4: now also J23.12
- net OUT_IGN5: now also J23.4
- net OUT_IGN6: now also J23.13
- net OUT_INJ1: now also J23.7
- net OUT_INJ2: now also J23.16
- net OUT_INJ3: now also J23.6
- net OUT_INJ4: now also J23.15
- net OUT_INJ5: now also J23.5
- net OUT_INJ6: now also J23.14
- net OUT_LS1: now also J23.10
- net OUT_LS2: now also J23.1
- net OUT_LS3: now also J23.8
- net OUT_LS4: now also J23.9
- net OUT_LS_HOT1: now also J25.34
- net OUT_LS_HOT2: now also J25.25
- net VR_DISCRETE+: now also J23.26
- net VR_DISCRETE-: now also J23.27
- net VR_MAX9924+: now also J23.18
- net VR_MAX9924-: now also J23.28
- net CAN2L: now reaches J23.19
- net CAN2L: now also M7.S1 (CANL)
- net CAN2H: now reaches J23.20
- net CAN2H: now also M7.S2 (CANH)
Other:
- moved on the sheet: J17, J21

Commit message: A
AAA
Connections:
- net +5VA: no longer J25.11, J25.12, J25.13, J25.2
- net CAN+: now also J25.29; no longer J25.30
- net CAN-: now also J25.30; no longer J25.31
- net EGT+: now also J25.18
- net EGT-: now also J25.19
- net IN_AUX1: now also J25.13; no longer J25.21
- net IN_BUTTON1: now also J25.12; no longer J25.1
- net IN_BUTTON2: now also J25.2; no longer J25.10
- net IN_CLT: now also J25.28; no longer J25.29
- net IN_FLEX: now also J25.11; no longer J25.19
- net IN_IAT: now also J25.27; no longer J25.28
- net IN_KNOCK_RAW: now also J25.20; no longer J25.27
- net IN_MAP: now also J25.21; no longer J25.20
- net IN_PPS1: now also J25.10; no longer J25.26
- net IN_TPS1: now also J25.1; no longer J25.18
- net WBO_Heater: now also J25.26
- net WBO_Ip: now also J25.32
- net WBO_Rtrim: now also J25.24
- net WBO_Un: now also J25.33
- net WBO_Vm: now also J25.31
