File: uaefi.kicad_sch (KiCad schematic)
At the start: 71 parts, among them J1 Conn_02x02_Odd_Even, J1 USB_B_Mini, J1 USB_C, J10 5569-16A2, J11 Conn_02x02_Odd_Even, J12 Conn_02x02_Odd_Even, J13 Conn_02x02_Odd_Even, J14 Conn_02x02_Odd_Even, J15 Conn_02x02_Odd_Even, J16 Conn_02x02_Odd_Even, J17 Conn_01x06, J17 Conn_02x02_Odd_Even, J18 Conn_02x02_Odd_Even, J19 Conn_02x02_Odd_Even, J2 5569-20A2, J20 Conn_02x02_Odd_Even, J21 Conn_02x02_Odd_Even, J22 Conn_02x02_Odd_Even, J23 2-6447232-3, J24 Conn_02x02_Odd_Even, J25 2-6447232-3, J3 5569-06A2, J4 5569-08A2, J5 5569-18A2, J5 Conn_01x05_Male, M1 Module-power_12and5V-0.3, M3 Module-knock-0.2, M3 Module-vr-discrete-0.5, M4 Module-vr-max9924-0.1, M5 Module-wbo-0.5, M6 Module:mega-mcu100/0.3, M7 Module-can-0.1, M8 Module-mega-mcu144-0.7, P3 Pad, P4 Pad, P5 Pad, P6 Pad, P7 Pad, P8 Pad, U4 JDY-33

Commit message: test
Parts:
- removed C3: 100n, hellen-one-common:C0603, symbol hellen-one-common:Cap
- removed F6 (x2): 12H1500D, hellen-one-common:PAD-1206-PAD, symbol hellen-one-common:Fuse-Pad-Pad
- removed J10: 5569-16A2, Connector_Molex:Molex_Mini-Fit_Jr_5569-16A2_2x08_P4.20mm_Horizontal, symbol Connector_Generic:Conn_02x08_Top_Bottom
- removed J2: 5569-20A2, Connector_Molex:Molex_Mini-Fit_Jr_5569-20A2_2x10_P4.20mm_Horizontal, symbol Connector_Generic:Conn_02x10_Top_Bottom
- removed J4: 5569-08A2, Connector_Molex:Molex_Mini-Fit_Jr_5569-08A2_2x04_P4.20mm_Horizontal, symbol Connector_Generic:Conn_02x04_Top_Bottom
- removed J5: 5569-18A2, Connector_Molex:Molex_Mini-Fit_Jr_5569-18A2_2x09_P4.20mm_Horizontal, symbol Connector_Generic:Conn_02x09_Top_Bottom
- removed M3: Module-knock-0.2, hellen-one-knock-0.2:knock, symbol hellen-one-knock-0.2:Module-knock-0.2
- removed M7: Module-can-0.1, hellen-one-can-0.1:can, symbol hellen-one-can-0.1:Module-can-0.1
- removed M8: Module-mega-mcu144-0.7, hellen-one-mega-mcu144-0.7:mega-mcu144, symbol Hellen 144:Module-mega-mcu144-0.7
- removed P7, P8: Pad, hellen-one-common:PAD-TH, symbol hellen-one-common:Pad
- removed R30: 0, hellen-one-common:R0603, symbol hellen-one-common:Res
- removed U4: JDY-33, kicad6-libraries:JDY-33, symbol JDY-33:JDY-33
Connections:
- net 12V_KEY: no longer F6.1
- net IN_KNOCK_RAW: no longer J25.20
- net IN_PPS1: no longer J25.10
- net IN_PPS2: no longer J25.15
- net OUT_DC1+: no longer J23.34
- net OUT_DC1-: no longer J23.33
- net OUT_DC2+: no longer J23.32
- net OUT_DC2-: no longer J23.31
- net OUT_IGN5: no longer J23.4
- net OUT_IGN6: no longer J23.13
- net OUT_INJ5: no longer J23.5
- net OUT_INJ6: no longer J23.14
- net OUT_LS3: no longer J23.8
- net OUT_LS4: no longer J23.9
- net CAN2H: no longer names the net of J23.20
- net CAN2L: no longer names the net of J23.19
- net EGT+: no longer names the net of J25.18
- net EGT-: no longer names the net of J25.19
- net EGT/SPI_CS: no longer names the net of M6.N9 (SPI3_CS_(PA15))
- no-connect marks 30 -> 27
Other:
- removed sheet DC Driver 1
- removed sheet DC Driver 2
- removed sheet EGT
- note removed: "3.5A MAX Solenoid load capable"
- note removed: "A"
- note removed: "B"
- note removed: "Bluetooth Module"
- note removed: "C"
- note removed: "D"
- note removed: "Pin 8 may be used for shielding VR signals"

Commit message: reset
Parts:
- added C3: 100n, hellen-one-common:C0603, symbol hellen-one-common:Cap
- added F6 (x2): 12H1500D, hellen-one-common:PAD-1206-PAD, symbol hellen-one-common:Fuse-Pad-Pad
- added J10: 5569-16A2, Connector_Molex:Molex_Mini-Fit_Jr_5569-16A2_2x08_P4.20mm_Horizontal, symbol Connector_Generic:Conn_02x08_Top_Bottom
- added J2: 5569-20A2, Connector_Molex:Molex_Mini-Fit_Jr_5569-20A2_2x10_P4.20mm_Horizontal, symbol Connector_Generic:Conn_02x10_Top_Bottom
- added J4: 5569-08A2, Connector_Molex:Molex_Mini-Fit_Jr_5569-08A2_2x04_P4.20mm_Horizontal, symbol Connector_Generic:Conn_02x04_Top_Bottom
- added J5: 5569-18A2, Connector_Molex:Molex_Mini-Fit_Jr_5569-18A2_2x09_P4.20mm_Horizontal, symbol Connector_Generic:Conn_02x09_Top_Bottom
- added M3: Module-knock-0.2, hellen-one-knock-0.2:knock, symbol hellen-one-knock-0.2:Module-knock-0.2
- added M7: Module-can-0.1, hellen-one-can-0.1:can, symbol hellen-one-can-0.1:Module-can-0.1
- added P7, P8: Pad, hellen-one-common:PAD-TH, symbol hellen-one-common:Pad
- added R30: 0, hellen-one-common:R0603, symbol hellen-one-common:Res
- added U4: JDY-33, kicad6-libraries:JDY-33, symbol JDY-33:JDY-33
Connections:
- net +12V: now also F6.1, F6.1, J4.8 (Pin_8)
- net +3.3VA: now also C3.2, M7.V2 (CAN_VIO), U4.12 (3V3)
- net +5VA: now also M3.E1 (V5A), M7.V1 (V5)
- net +5VP: now also J10.3 (Pin_3), J10.4 (Pin_4), J2.1 (Pin_1), J2.2 (Pin_2)
- net 12V_KEY: now also F6.1, J4.7 (Pin_7)
- net ADC3: now also R30.2
- net CAN+: now also J10.7 (Pin_7)
- net CAN-: now also J10.8 (Pin_8)
- net GND: now also C3.1, J2.8 (Pin_8), J4.3 (Pin_3), J4.4 (Pin_4), M3.E2 (GND), M7.E1 (GND), U4.13 (GND)
- net GNDA: now also J10.11 (Pin_11), J10.12 (Pin_12), J2.11 (Pin_11), J2.12 (Pin_12), J2.13 (Pin_13)
- net IN_AUX1: now also J10.1 (Pin_1)
- net IN_AUX2: now also J2.3 (Pin_3)
- net IN_AUX3: now also J2.15 (Pin_15)
- net IN_BUTTON1: now also J10.2 (Pin_2)
- net IN_BUTTON2: now also J10.10 (Pin_10)
- net IN_BUTTON3: now also J2.9 (Pin_9)
- net IN_CLT: now also J10.16 (Pin_16)
- net IN_FLEX: now also J10.5 (Pin_5)
- net IN_HALL1: now also J2.5 (Pin_5)
- net IN_HALL2: now also J2.6 (Pin_6)
- net IN_HALL3: now also J2.7 (Pin_7)
- net IN_IAT: now also J10.15 (Pin_15)
- net IN_KNOCK_RAW: now also J25.20, J10.14 (Pin_14), M3.W1 (IN_KNOCK)
- net IN_MAP: now also J10.9 (Pin_9)
- net IN_PPS1: now also J25.10, J10.6 (Pin_6)
- net IN_PPS2: now also J25.15, J2.4 (Pin_4)
- net IN_TPS1: now also J10.13 (Pin_13)
- net IN_TPS2: now also J2.14 (Pin_14)
- net OUT_DC1+: now also J23.34, J4.5 (Pin_5)
- net OUT_DC1-: now also J23.33, J4.1 (Pin_1)
- net OUT_DC2+: now also J23.32, J4.6 (Pin_6)
- net OUT_DC2-: now also J23.31, J4.2 (Pin_2)
- net OUT_IGN1: now also J5.15 (Pin_15)
- net OUT_IGN2: now also J5.14 (Pin_14)
- net OUT_IGN3: now also J5.12 (Pin_12)
- net OUT_IGN4: now also J5.11 (Pin_11)
- net OUT_IGN5: now also J23.4, J5.13 (Pin_13)
- net OUT_IGN6: now also J23.13, J5.10 (Pin_10)
- net OUT_INJ1: now also J5.6 (Pin_6)
- net OUT_INJ2: now also J5.5 (Pin_5)
- net OUT_INJ3: now also J5.4 (Pin_4)
- net OUT_INJ4: now also J5.3 (Pin_3)
- net OUT_INJ5: now also J23.5, J5.2 (Pin_2)
- net OUT_INJ6: now also J23.14, J5.1 (Pin_1)
- net OUT_LS1: now also J5.7 (Pin_7)
- net OUT_LS2: now also J5.18 (Pin_18)
- net OUT_LS3: now also J23.8, J5.17 (Pin_17)
- net OUT_LS4: now also J23.9, J5.16 (Pin_16)
- net OUT_LS_HOT1: now also J5.9 (Pin_9)
- net OUT_LS_HOT2: now also J5.8 (Pin_8)
- net VREF1: now also M3.W2 (VREF)
- net VR_DISCRETE+: now also J2.18 (Pin_18)
- net VR_DISCRETE-: now also J2.19 (Pin_19)
- net VR_MAX9924+: now also J2.16 (Pin_16)
- net VR_MAX9924-: now also J2.17 (Pin_17)
- net at M6.E6 (SPI2_CS_/_CAN2_RX_(PB12)): now also M7.V6 (CAN_RX)
- net at M6.E7 (SPI2_SCK_/_CAN2_TX_(PB13)): now also M7.V5 (CAN_TX)
- net at M6.N13 (UART2_TX_(PD5)): now also P8.1 (Pin_1), U4.2 (RXD)
- net at M6.N14 (UART2_RX_(PD6)): now also P7.1 (Pin_1), U4.1 (TXD)
- net EGT/SPI_CS: now reaches M6.N9 (SPI3_CS_(PA15))
- net CAN2L: now reaches J23.19
- net CAN2L: now also M7.S1 (CANL)
- net CAN2H: now reaches J23.20
- net CAN2H: now also M7.S2 (CANH)
- net EGT+: now reaches J25.18
- net EGT+: now also J2.10 (Pin_10)
- net EGT-: now reaches J25.19
- net EGT-: now also J2.20 (Pin_20)
- new net DC Driver 1/PWR: F6.2
- new net DC Driver 2/PWR: F6.2
- new net IN_KNOCK: M3.E3 (OUT_KNOCK), R30.1
- no-connect marks 27 -> 30
Other:
- added sheet DC Driver 1 (DC_MOTOR_0.1.kicad_sch)
- added sheet DC Driver 2 (DC_MOTOR_0.1.kicad_sch)
- added sheet EGT (egt.kicad_sch)
- note added: "3.5A MAX Solenoid load capable"
- note added: "A"
- note added: "B"
- note added: "Bluetooth Module"
- note added: "C"
- note added: "D"
- note added: "Pin 8 may be used for shielding VR signals"

Commit message: a
a
Parts:
- J23, J25: LCSC (none) -> C574788
- J5: LCSC (none) -> C474923
Changed lines of the file:
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@@
+			)
+		)
+		(property "LCSC" "C574788"
+			(at -12.7 297.18 0)
+			(effects
+				(font
+					(size 1.27 1.27)
+				)
+				(hide yes)
 			)
 		)
@@
 			)
 		)
+		(property "LCSC" "C574788"
+			(at -13.97 189.23 0)
+			(effects
+				(font
+					(size 1.27 1.27)
+				)
+				(hide yes)
+			)
+		)
 		(pin "20"
 		)
@@
 			(at 236.22 302.26 0)
 			(effects
+				(font
+					(size 1.27 1.27)
+				)
+				(hide yes)
+			)
+		)
+		(property "LCSC" "C474923"
+			(at 236.22 302.26 0)
+			(effects
