File: DC_MOTOR_0.1.kicad_sch (KiCad schematic)
At the start: 17 parts, among them P15 Pad, P17 Pad

Commit message: test
Parts:
- removed C? (x10): 10u, hellen-one-common:C0805, symbol hellen-one-common:Cap
- removed C?: 100n, hellen-one-common:C0603, symbol hellen-one-common:Cap
- removed C? (x2): 10n, hellen-one-common:C0603, symbol hellen-one-common:Cap
- removed P15, P17: Pad, hellen-one-common:PAD-TH, symbol hellen-one-common:Pad
- removed R?: 4.7k, hellen-one-common:R0603, symbol hellen-one-common:Res
- removed U?: TLE9201SG, Package_SO:Infineon_PG-DSO-12-11, symbol chips:TLE9201SG
Connections:
- no-connect marks 1 -> 0

Commit message: reset
Parts:
- added C? (x10): 10u, hellen-one-common:C0805, symbol hellen-one-common:Cap
- added C?: 100n, hellen-one-common:C0603, symbol hellen-one-common:Cap
- added C? (x2): 10n, hellen-one-common:C0603, symbol hellen-one-common:Cap
- added P15, P17: Pad, hellen-one-common:PAD-TH, symbol hellen-one-common:Pad
- added R?: 4.7k, hellen-one-common:R0603, symbol hellen-one-common:Res
- added U?: TLE9201SG, Package_SO:Infineon_PG-DSO-12-11, symbol chips:TLE9201SG
Connections:
- new net 3V3: R?.2, U?.2 (VSO)
- new net DIR: P15.1 (Pin_1), U?.1 (DIR)
- new net DIS: R?.1, U?.11 (DIS)
- new net GND: C?.1, C?.1, C?.1, C?.1, C?.1, C?.1, C?.1, C?.1, C?.1, C?.1, C?.1, C?.1, C?.1, U?.10 (SCK), U?.13 (GND), U?.6 (GND), U?.8 (SI), U?.9 (CSN)
- new net OUT+: C?.2, U?.7 (OUT2)
- new net OUT-: C?.2, U?.5 (OUT1)
- new net PWM: P17.1 (Pin_1), U?.12 (PWM)
- new net PWR: C?.2, C?.2, C?.2, C?.2, C?.2, C?.2, C?.2, C?.2, C?.2, C?.2, C?.2, U?.4 (VS)
- no-connect marks 0 -> 1
