File: MAP.kicad_sch (KiCad schematic)
At the start: 2 parts, among them U3 MPX4/MPXH6400_MAP

Commit message: a
a
Parts:
- U3: LCSC (none) -> C511770
Changed lines of the file:
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@@
+			)
+		)
+		(property "LCSC" "C511770"
+			(at 146.05 90.17 0)
+			(effects
+				(font
+					(size 1.27 1.27)
+				)
+				(hide yes)
 			)
 		)
